File: FlipperZeroESP32/FlipperZeroESP32.kicad_pcb (KiCad board)
At the start: 2 copper layers, 85 x 45 mm, 31 parts, among them J1 Conn_Flipper_L, J2 Conn_Flipper_R, J3 USB C connector, J4 Breakout_1, J5 Breakout_2, Q1 2N7002, Q2 2N7002, SW1 RESET_BTN, SW2 FLASH_BTN, U1 AMS1117-3.3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

Commit message: Start new hardware design
Parts:
- added G***: LOGO, Flipper-Zero-ESP32-GPIO-Board:Raven_Logo, F.Cu at (145.0, 106.4)
- moved C5 116.8 mm to (181.6, 134.1)
- moved C6 116.6 mm to (181.6, 131.1)
- moved Q2 103.2 mm to (181.5, 127.5)
- moved Q1 103.1 mm to (181.5, 124.0)
- moved R1 103.0 mm to (173.5, 119.0), turned to -90 degrees
- moved R2 103.0 mm to (173.5, 113.0), turned to 90 degrees
- moved C1 101.6 mm to (166.5, 111.0), turned to 180 degrees
- moved R7 96.7 mm to (167.0, 126.0), turned to -90 degrees
- moved R6 96.4 mm to (167.0, 131.5), turned to -90 degrees
- moved C4 91.5 mm to (156.0, 115.5), turned to 180 degrees
- moved C2 91.1 mm to (156.0, 121.5), turned to 180 degrees
- moved C3 91.1 mm to (156.0, 118.5), turned to 180 degrees
- moved R5 65.5 mm to (133.0, 107.5), turned to -90 degrees
- moved R4 51.3 mm to (121.2, 132.5), turned to 180 degrees
- moved C7 50.7 mm to (115.6, 132.5), turned to 180 degrees
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- renumbered He to H1
Connections:
- J2 pad 17: unconnected-(J2-Pin_17-Pad17) -> GND
- J2 pad 18: unconnected-(J2-Pin_18-Pad18) -> GND
- J4 pad 6: unconnected-(J4-Pin_6-Pad6) -> GND
- J4 pad 7: unconnected-(J4-Pin_7-Pad7) -> GND
Routing:
- net RST: track 0.00 -> 129.0 mm, vias 0 -> 1
- net +5V: track 0.00 -> 125.9 mm, vias 0 -> 1
- net TXD0: track 0.00 -> 107.1 mm, vias 0 -> 4
- net RXD0: track 0.00 -> 101.9 mm, vias 0 -> 4
- net IO0: track 0.00 -> 84.2 mm, vias 0 -> 1
- net DTR: track 0.00 -> 76.9 mm, vias 0 -> 2
- net RTS: track 0.00 -> 75.2 mm, vias 0 -> 2
- net IO1: track 0.00 -> 69.0 mm
- net IO2: track 0.00 -> 64.0 mm, vias 0 -> 1
- net IO17: track 0.00 -> 51.3 mm, vias 0 -> 2
- net IO18: track 0.00 -> 47.5 mm
- net +3V3: track 0.00 -> 35.7 mm, vias 0 -> 12
- net IO7: track 0.00 -> 33.2 mm, vias 0 -> 1
- net GND: track 0.00 -> 32.1 mm, vias 0 -> 10
- net IO11: track 0.00 -> 30.4 mm, vias 0 -> 1
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- added copper zone on In2.Cu, net +3V3
- added copper zone on B.Cu, net GND
- added copper zone on F.Cu, net GND
- added copper zone on In1.Cu, net GND
Other:
- copper layers 2 -> 4
- board text added: "+3V3"
- board text added: "+5V"
- board text added: "DTR"
- board text added: "GND"
- board text added: "IO1"
- board text added: "IO10"
- board text added: "IO11"
- board text added: "IO12"
- board text added: "IO13"
- board text added: "IO14"
- board text added: "IO15"
- board text added: "IO16"
- board text added: "IO17"
- board text added: "IO18"
- board text added: "IO2"
- board text added: "IO21"
- board text added: "IO35"
- board text added: "IO36"
- board text added: "IO37"
- board text added: "IO7"
- board text added: "IO8"
- board text added: "IO9"
- board text added: "RST"
- board text added: "RTS"
- board text added: "RXD0"
- board text added: "TCK"
- board text added: "TDI"
- board text added: "TDO"
- board text added: "TMS"
- board text added: "TXD0"
