File: FlipperZeroESP32/FlipperZeroESP32.kicad_sch (KiCad schematic)
At the start: 31 parts, among them J1 Conn_Flipper_L, J2 Conn_Flipper_R, J3 USB C connector, J4 Breakout_1, J5 Breakout_2, Q1 2N7002, Q2 2N7002, SW1 RESET_BTN, SW2 FLASH_BTN, U1 AMS1117-3.3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

Commit message: Start new hardware design
Connections:
- net GND: now also J2.17 (Pin_17), J2.18 (Pin_18), J4.6 (Pin_6), J4.7 (Pin_7)
Changed lines of the file:
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@@
   (junction (at 190.5 152.4) (diameter 0) (color 0 0 0 0)
   )
+  (junction (at 121.92 76.2) (diameter 0) (color 0 0 0 0)
+  )
   (junction (at 251.46 27.94) (diameter 0) (color 0 0 0 0)
   )
@@
   (junction (at 109.22 48.26) (diameter 0) (color 0 0 0 0)
   )
+  (junction (at 162.56 53.34) (diameter 0) (color 0 0 0 0)
+  )
   (junction (at 50.8 48.26) (diameter 0) (color 0 0 0 0)
   )
@@
   (junction (at 149.86 55.88) (diameter 0) (color 0 0 0 0)
   )
+  (junction (at 149.86 53.34) (diameter 0) (color 0 0 0 0)
+  )
   (junction (at 200.66 76.2) (diameter 0) (color 0 0 0 0)
   )
@@
   (junction (at 149.86 27.94) (diameter 0) (color 0 0 0 0)
   )
+  (junction (at 106.68 76.2) (diameter 0) (color 0 0 0 0)
+  )
   (junction (at 129.54 124.46) (diameter 0) (color 0 0 0 0)
   )
@@
     (stroke (width 0) (type default))
   )
+  (wire (pts (xy 96.52 66.04) (xy 96.52 76.2))
+    (stroke (width 0) (type default))
+  )
   (wire (pts (xy 215.9 53.34) (xy 223.52 53.34))
     (stroke (width 0) (type default))
@@
     (stroke (width 0) (type default))
   )
+  (wire (pts (xy 96.52 66.04) (xy 109.22 66.04))
+    (stroke (width 0) (type default))
+  )
   (wire (pts (xy 162.56 40.64) (xy 165.1 40.64))
     (stroke (width 0) (type default))
@@
     (stroke (width 0) (type default))
   )
+  (wire (pts (xy 162.56 50.8) (xy 162.56 53.34))
+    (stroke (width 0) (type default))
+  )
   (wire (pts (xy 193.04 134.62) (xy 195.58 134.62))
     (stroke (width 0) (type default))
@@
     (stroke (width 0) (type default))
   )
+  (wire (pts (xy 149.86 50.8) (xy 149.86 53.34))
+    (stroke (width 0) (type default))
+  )
   (wire (pts (xy 121.92 27.94) (xy 121.92 30.48))
     (stroke (width 0) (type default))
@@
     (stroke (width 0) (type default))
   )
-  (wire (pts (xy 106.68 66.04) (xy 109.22 66.04))
-    (stroke (width 0) (type default))
-  )
   (wire (pts (xy 121.92 68.58) (xy 124.46 68.58))
     (stroke (width 0) (type default))
@@
     (stroke (width 0) (type default))
   )
+  (wire (pts (xy 134.62 63.5) (xy 134.62 76.2))
+    (stroke (width 0) (type default))
+  )
   (wire (pts (xy 231.14 147.32) (xy 248.92 147.32))
     (stroke (width 0) (type default))
@@
     (stroke (width 0) (type default))
   )
-  (wire (pts (xy 121.92 63.5) (xy 124.46 63.5))
+  (wire (pts (xy 121.92 63.5) (xy 134.62 63.5))
     (stroke (width 0) (type default))
   )
@@
     (stroke (width 0) (type default))
   )
+  (wire (pts (xy 96.52 76.2) (xy 106.68 76.2))
+    (stroke (width 0) (type default))
+  )
   (wire (pts (xy 71.12 35.56) (xy 71.12 38.1))
     (stroke (width 0) (type default))
@@
     (stroke (width 0) (type default))
   )
+  (wire (pts (xy 134.62 76.2) (xy 121.92 76.2))
+    (stroke (width 0) (type default))
+  )
